Commit message: Edit base position

File: six_dof_cam_description/urdf/base/base.xacro (robot description, xacro)
@@ -2,6 +2,6 @@
 <robot xmlns:xacro="http://ros.org/wiki/xacro">
 	<xacro:include filename="$(find six_dof_cam_description)/urdf/base/base.gazebo.xacro"/>
-	<!--<xacro:property name="M_PI" value="3.1415926535897931" />-->
-	<!--<xacro:property name="velocity_scale_factor" value="1.0"/>-->
+	<xacro:property name="M_PI" value="3.1415926535897931" />
+	<xacro:property name="velocity_scale_factor" value="1.0"/>
 	<xacro:macro name="base" params="parent *joint_origin">
 		<joint name="base_joint" type="fixed">
@@ -15,4 +15,5 @@
 					<box size="0.1 0.1 0.1"/>
 				</geometry>
+				<origin rpy="0 0 0" xyz="0.05 0 0.05"/>
 			</visual>
 			<collision>
@@ -20,4 +21,5 @@
 					<box size="0.1 0.1 0.1"/>
 				</geometry>
+				<origin rpy="0 0 0" xyz="0.05 0 0.05"/>
 			</collision>
 			<inertial>

File: six_dof_cam_description/urdf/camera/camera.gazebo.xacro (robot description, xacro)
@@ -1,4 +1,5 @@
 <?xml version="1.0"?>
 <robot xmlns:xacro="http://ros.org/wiki/xacro">
+	<xacro:property name="M_PI" value="3.1415926535897931" />
 	<xacro:macro name="camera_gazebo">
 		<gazebo reference="camera_link">
@@ -10,5 +11,5 @@
 				<camera name="left">
 					<pose>0 0.03 0 0 0 0</pose>
-					<horizontal_fov>1.3962634</horizontal_fov>
+					<horizontal_fov>${M_PI / 180 * 110}</horizontal_fov>
 					<image>
 						<width>800</width>
@@ -28,5 +29,5 @@
 				<camera name="right">
 					<pose>0 -0.03 0 0 0 0</pose>
-					<horizontal_fov>1.3962634</horizontal_fov>
+					<horizontal_fov>${M_PI / 180 * 110}</horizontal_fov>
 					<image>
 						<width>800</width>
@@ -61,41 +62,4 @@
 			</sensor>
 		</gazebo>
-<!--
-			<sensor type="camera" name="camera1">
-			<update_rate>60.0</update_rate>
-			<camera name="head">
-			<horizontal_fov>1.3962634</horizontal_fov>
-			<image>
-			<width>800</width>
-			<height>800</height>
-			<format>R8G8B8</format>
-			</image>
-			<clip>
-			<near>0.02</near>
-			<far>300</far>
-			</clip>
-			<noise>
-			<type>gaussian</type>
-			<mean>0.0</mean>
-			<stddev>0.007</stddev>
-			</noise>
-			</camera>
-			<plugin name="camera_controller" filename="libgazebo_ros_camera.so">
-			<alwaysOn>true</alwaysOn>
-			<updateRate>0.0</updateRate>
-			<cameraName>six_dof_cam/camera1</cameraName>
-			<imageTopicName>image_raw</imageTopicName>
-			<cameraInfoTopicName>camera_info</cameraInfoTopicName>
-			<frameName>camera_link</frameName>
-			<hackBaseline>0.07</hackBaseline>
-			<distortionK1>0.0</distortionK1>
-			<distortionK2>0.0</distortionK2>
-			<distortionK3>0.0</distortionK3>
-			<distortionT1>0.0</distortionT1>
-			<distortionT2>0.0</distortionT2>
-			</plugin>
-			</sensor>
-		</gazebo>
--->
 	</xacro:macro>
 </robot>

File: six_dof_cam_description/urdf/six_dof_cam.xacro (robot description, xacro)
@@ -9,5 +9,5 @@
 	<link name="world"/>
 	<xacro:base parent="world">
-		<origin xyz="0 0 0.05" rpy="0 0 0"/>
+		<origin xyz="0 0 0" rpy="0 0 0"/>
 	</xacro:base>
 	<xacro:linear_actuator prefix="x" parent="base_link">
