Commit message: Edit position offset

File: six_dof_cam_description/urdf/six_dof_cam.xacro (robot description, xacro)
@@ -12,5 +12,5 @@
 	</xacro:base>
 	<xacro:linear_actuator prefix="x" parent="base_link">
-		<origin xyz="0 0 1" rpy="0 0 0"/>
+		<origin xyz="0 0 0" rpy="0 0 0"/>
 		<axis xyz="1 0 0"/>
 	</xacro:linear_actuator>
